File: Main_DIP_Controller.kicad_pcb (KiCad board)
At the start: 4 copper layers, 100 x 100 mm, 50 parts, among them J1 Switch_Control, J10 Vin_-, J11 Conn_01x02, J12 Vsens, J13 Vin+, J2 2.1-5.5 DC, J3 +5V, J4 AnalogIO, J5 +12V, J6 VsensJMP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

Commit message: Finish parts placement
Parts:
- P1: footprint Eoshi-chan:Eoshi-chan_logo_10x10 -> Eoshi-chan_v2:Eoshi-chan-v2_13x13
- moved H3 272.5 mm to (55.0, 55.0)
- moved P1 267.7 mm to (68.0, 136.0)
- moved H4 267.1 mm to (55.0, 140.0)
- moved J3 240.1 mm to (72.4, 118.1), turned to 90 degrees
- moved J8 239.8 mm to (72.4, 92.7), turned to 90 degrees
- moved U1 237.4 mm to (92.7, 123.9), turned to 180 degrees
- moved RV1 229.8 mm to (84.6, 95.2), turned to 90 degrees
- moved Q1 210.6 mm to (112.3, 89.7), turned to 180 degrees
- moved H2 210.3 mm to (117.0, 55.0)
- moved HS1 209.7 mm to (90.2, 128.4), turned to 180 degrees
- moved C9 209.1 mm to (74.3, 109.7), turned to 180 degrees
- moved H1 209.0 mm to (117.0, 140.0)
- moved C3 207.6 mm to (79.5, 123.9), turned to -90 degrees
- moved J11 201.1 mm to (116.8, 68.6), turned to 90 degrees
- moved C4 197.3 mm to (73.7, 125.5), turned to -90 degrees
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Other:
- board size 100 x 100 mm -> 72 x 95 mm
